Commit message: Seperate dependency from gripper.
The dependency from the gripper was removed to allow easier
transition between ros distros.

File: prbt_moveit_config/config/prbt.srdf.xacro (robot description, xacro)
@@ -2,5 +2,6 @@
 <robot name="prbt" xmlns:xacro="http://www.ros.org/wiki/xacro">
   <!-- parameter -->
-  <xacro:arg name="has_gripper" default="false"/>
+  <xacro:arg name="gripper" default=""/>
+  <xacro:property name="gripper" value="$(arg gripper)"/>
   <xacro:arg name="prefix" default="prbt_"/>
   <!--VIRTUAL JOINT: Purpose: this element defines a virtual joint between a robot link and an
@@ -11,7 +12,6 @@
   <xacro:prbt_manipulator prefix="$(arg prefix)"/>
   <!-- has gripper -->
-  <xacro:if value="$(arg has_gripper)">
-    <xacro:include filename="$(find prbt_moveit_config)/config/prbt_pg70.srdf.xacro" />
-    <xacro:prbt_pg70 prefix="$(arg prefix)"/>
-  </xacro:if>
+  <xacro:unless value="${not gripper}">
+    <xacro:include filename="$(find prbt_${gripper}_support)/config/${gripper}.srdf.xacro" />
+  </xacro:unless>
 </robot>

File: prbt_support/urdf/prbt.xacro (robot description, xacro)
@@ -18,13 +18,13 @@
   <xacro:include filename="$(find prbt_support)/urdf/prbt_macro.xacro" />
   <!-- gripper -->
-  <xacro:arg name="has_gripper" default="false"/>
+  <xacro:arg name="gripper" default=""/>
+  <xacro:property name="gripper" value="$(arg gripper)"/>
   <!-- TCP Offset -->
-  <xacro:unless value="$(arg has_gripper)">
+  <xacro:if value="${not gripper}">
     <xacro:arg name="tcp_offset_xyz" default="0 0 0"/>
     <xacro:arg name="tcp_offset_rpy" default="0 0 0"/>
-  </xacro:unless>
-  <xacro:if value="$(arg has_gripper)">
-    <xacro:arg name="tcp_offset_xyz" default="0 0 0.1"/>
-    <xacro:arg name="tcp_offset_rpy" default="0 0 ${-pi*3/4.}"/>
+  </xacro:if>
+  <xacro:if value="${gripper != ''}">
+    <xacro:include filename="$(find prbt_${gripper}_support)/config/${gripper}_tcp_offset.xacro" />
   </xacro:if>
   <!-- instantiate the robot -->
@@ -37,19 +37,7 @@
   </joint>
   <link name="$(arg robot_prefix)tcp" />
-  <xacro:if value="$(arg has_gripper)">
-    <!-- Load pg70 gripper macro -->
-    <xacro:include filename="$(find schunk_description)/urdf/pg70/pg70.urdf.xacro" />
-    <!-- name of the gripper -->
-    <xacro:arg name="gripper_name" default="$(arg robot_prefix)gripper"/>
-    <!-- instantiate the gripper -->
-    <xacro:schunk_pg70 parent="$(arg robot_prefix)flange" name="$(arg gripper_name)" has_podest="false">
-      <origin xyz="0 0 0.0171" rpy="0 0 ${-pi*3/4.}" />
-    </xacro:schunk_pg70>
-    <!-- Add gripper brackets -->
-    <xacro:include filename="$(find prbt_support)/urdf/simple_gripper_brackets.urdf.xacro" />
-    <xacro:simple_gripper_brackets
-        gripper_name="$(arg gripper_name)"
-        parent_left="$(arg gripper_name)_finger_left_link"
-        parent_right="$(arg gripper_name)_finger_right_link"/>
+  <!-- If gripper given then... -->
+  <xacro:if value="${gripper != ''}">
+    <xacro:include filename="$(find prbt_${gripper}_support)/urdf/${gripper}.urdf.xacro" />
   </xacro:if>
 </robot>
