Commit message: support: move constant defs inside macro def
This allows xacro to namespace the constants and avoids collisions with other xacros.

File: prbt_support/urdf/prbt_macro.xacro (robot description, xacro)
@@ -13,13 +13,13 @@
 -->
 <robot xmlns:xacro="http://www.ros.org/wiki/xacro">
-  <!-- Height of Foot -->
-  <xacro:property name="L0" value="0.2604" />
-  <!-- Length of the first connector -->
-  <xacro:property name="L1" value="0.3500" />
-  <!-- Length of the second connector -->
-  <xacro:property name="L2" value="0.3070" />
-  <!-- Distance last joint to flange -->
-  <xacro:property name="L3" value="0.0840" />
   <xacro:macro name="prbt" params="prefix">
+    <!-- Height of Foot -->
+    <xacro:property name="L0" value="0.2604" />
+    <!-- Length of the first connector -->
+    <xacro:property name="L1" value="0.3500" />
+    <!-- Length of the second connector -->
+    <xacro:property name="L2" value="0.3070" />
+    <!-- Distance last joint to flange -->
+    <xacro:property name="L3" value="0.0840" />
     <!-- robot foot link -->
     <link name="${prefix}base_link">

Commit message: Add inertial tag to base_link
The `<inertial>` tag is required to use the model with MoveIt! and Gazebo.
The provided `mass value` is a rough guess.

Otherwise `gazebo_ros_control` fails with the following error:
```shell
[ INFO] [1536068104.372075788]: gazebo_ros_control plugin is waiting for model URDF in parameter [/robot_description] on the ROS param server.
[ERROR] [1536068104.507384025]: This robot has a joint named "prbt_joint_1" which is not in the gazebo model.
[FATAL] [1536068104.507615381]: Could not initialize robot simulation interface
```

File: prbt_support/urdf/prbt_macro.xacro (robot description, xacro)
@@ -24,4 +24,8 @@
     <!-- robot foot link -->
     <link name="${prefix}base_link">
+      <inertial>
+        <mass value="5"/>
+        <inertia ixx="0"  ixy="0"  ixz="0" iyy="0" iyz="0" izz="0" />
+      </inertial>
       <visual>
         <origin xyz="0 0 0" rpy="0 0 0" />

Commit message: move interial tensors into center-of-mass system
* specify center of mass for the links
* reduce inertial tensor accordingly

File: prbt_support/urdf/prbt_macro.xacro (robot description, xacro)
@@ -54,5 +54,6 @@
       <inertial>
         <mass value="7.1"/>
-        <inertia ixx="5.84e-2"  ixy="-1.1e-5"  ixz="6.5e-5" iyy="4.84e-2" iyz="-2.8e-4" izz="2.34e-2" />
+        <origin xyz="0 -0.026 -0.051" />
+        <inertia ixx="3.53e-2" ixy="0" ixz="0" iyy="3.01e-2" iyz="9.04e-3" izz="1.87e-2" />
       </inertial>
       <visual>
@@ -93,5 +94,6 @@
       <inertial>
         <mass value="1.7"/>
-        <inertia ixx="1.12e-1"  ixy="-1.7e-6"  ixz="-8e-7" iyy="3.40e-2" iyz="-3.87e-2" izz="8.17e-2" />
+        <origin xyz="0 0.162 0.134" />
+        <inertia ixx="3.58e-2"  ixy="0"  ixz="0" iyy="3.22e-3" iyz="-1.45e-3" izz="3.66e-2" />
       </inertial>
       <visual name="first">
@@ -126,5 +128,6 @@
       <inertial>
         <mass value="4.8"/>
-        <inertia ixx="3.32e-2"  ixy="2.7e-6"  ixz="-3.3e-6" iyy="1.43e-2" iyz="2.3e-4" izz="2.54e-2" />
+        <origin xyz="0 0.043 -0.027" />
+        <inertia ixx="2.06e-2" ixy="0" ixz="0" iyy="1.08e-2" iyz="-5.36e-3" izz="1.63e-2" />
       </inertial>
       <visual>
@@ -165,5 +168,6 @@
       <inertial>
         <mass value="0.9"/>
-        <inertia ixx="4.7e-2"  ixy="-1.1e-6"  ixz="-9.8e-6" iyy="4.15e-2" iyz="1.35e-2" izz="6.63e-3" />
+        <origin xyz="0 -0.061 0.204" />
+        <inertia ixx="6.79e-3" ixy="0" ixz="0" iyy="4.91e-3" iyz="2.67e-3" izz="3.40e-3" />
       </inertial>
       <visual>
@@ -198,5 +202,6 @@
       <inertial>
         <mass value="2.6"/>
-        <inertia ixx="1.13e-2"  ixy="6.0e-5"  ixz="-2.7e-5" iyy="8.68e-3" iyz="7.9e-5" izz="5.10e-3" />
+        <origin xyz="-0.001 0.021 -0.032" />
+        <inertia ixx="7.37e-3" ixy="4.78e-6" ixz="6.00e-5" iyy="5.87e-3" iyz="-1.71e-3" izz="3.96e-3" />
       </inertial>
       <visual>
@@ -249,5 +254,6 @@
     <link name="${prefix}flange">
       <inertial>
-        <mass value="0.1" />
+        <mass value="0.02" />
+        <origin xyz="0 0 0" />
         <inertia ixx="0" ixy="0" ixz="0" iyy="0" iyz="0" izz="0" />
       </inertial>

Commit message: Relax joint limits. Fixes #82
Replace the radian values for the position limits (they have been rounded too roughly).

File: prbt_support/urdf/prbt_macro.xacro (robot description, xacro)
@@ -47,5 +47,5 @@
       <child link="${prefix}link_1"/>
       <axis xyz="0 0 1"/>
-      <limit effort="370" velocity="1.57" lower="-2.967" upper="2.967"/>
+      <limit effort="370" velocity="1.57" lower="-2.96706" upper="2.96706"/>
       <dynamics damping="15.0" friction="11" />
     </joint>
@@ -88,5 +88,5 @@
       <child link="${prefix}link_2"/>
       <axis xyz="0 0 1"/>
-      <limit effort="370" velocity="1.57" lower="-2.531" upper="2.531"/>
+      <limit effort="370" velocity="1.57" lower="-2.53073" upper="2.53073"/>
       <dynamics damping="12.0" friction="10.0" />
     </joint>
@@ -122,5 +122,5 @@
       <child link="${prefix}link_3"/>
       <axis xyz="0 0 1"/>
-      <limit effort="176" velocity="1.57" lower="-2.356" upper="2.356"/>
+      <limit effort="176" velocity="1.57" lower="-2.35620" upper="2.35620"/>
       <dynamics damping="4.5" friction="4.5" />
     </joint>
@@ -162,5 +162,5 @@
       <child link="${prefix}link_4"/>
       <axis xyz="0 0 1" />
-      <limit effort="176" velocity="1.57" lower="-2.967" upper="2.967"/>
+      <limit effort="176" velocity="1.57" lower="-2.96706" upper="2.96706"/>
       <dynamics damping="4.2" friction="3.8" />
     </joint>
@@ -196,5 +196,5 @@
       <child link="${prefix}link_5"/>
       <axis xyz="0 0 1" />
-      <limit effort="41.6" velocity="1.57" lower="-2.967" upper="2.967" />
+      <limit effort="41.6" velocity="1.57" lower="-2.96706" upper="2.96706" />
       <dynamics damping="1.5" friction="3.5" />
     </joint>
@@ -248,5 +248,5 @@
       <child link="${prefix}flange"/>
       <axis xyz="0 0 1" />
-      <limit effort="20.1" velocity="1.57" lower="-3.124" upper="3.124" />
+      <limit effort="20.1" velocity="1.57" lower="-3.12414" upper="3.12414" />
       <dynamics damping="4.5" friction="7.0" />
     </joint>
