Commit message: Enable prbt model to be used in combination with Gazebo

File: prbt_support/urdf/prbt.xacro (robot description, xacro)
@@ -30,4 +30,9 @@
   <!-- instantiate the robot -->
   <xacro:prbt prefix="$(arg robot_prefix)" />
+  <link name="world"/>
+  <joint name="fixed" type="fixed">
+    <parent link="world"/>
+    <child link="$(arg robot_prefix)base_link"/>
+  </joint>
   <!-- TCP -->
   <joint name="$(arg robot_prefix)fixed_joint_tcp" type="fixed">

File: prbt_support/urdf/prbt_macro.xacro (robot description, xacro)
@@ -24,4 +24,8 @@
     <!-- robot foot link -->
     <link name="${prefix}base_link">
+        <inertial>
+          <mass value="2.4"/>
+          <inertia ixx="0"  ixy="0"  ixz="0" iyy="0" iyz="0" izz="0" />
+        </inertial>
       <visual>
         <origin xyz="0 0 0" rpy="0 0 0" />
@@ -49,7 +53,6 @@
     <link name="${prefix}link_1">
       <inertial>
-        <origin xyz="-0.00014 0.02783 0.05093" rpy="0 0 0"/>
         <mass value="7.1"/>
-        <inertia ixx="0"  ixy="0"  ixz="0" iyy="0" iyz="0" izz="0" />
+        <inertia ixx="5.84e-2"  ixy="-1.1e-5"  ixz="6.5e-5" iyy="4.84e-2" iyz="-2.8e-4" izz="2.34e-2" />
       </inertial>
       <visual>
@@ -89,7 +92,6 @@
     <link name="${prefix}link_2">
       <inertial>
-        <origin xyz="0.00001 0.16907 0.02464" rpy="0 0 0"/>
-        <mass value="2.4"/>
-        <inertia ixx="0"  ixy="0"  ixz="0" iyy="0" iyz="0" izz="0" />
+        <mass value="1.7"/>
+        <inertia ixx="1.12e-1"  ixy="-1.7e-6"  ixz="-8e-7" iyy="3.40e-2" iyz="-3.87e-2" izz="8.17e-2" />
       </inertial>
       <visual name="first">
@@ -123,7 +125,6 @@
     <link name="${prefix}link_3">
       <inertial>
-        <origin xyz="-0.0001 0.04395 -0.02798" rpy="0 0 0"/>
-        <mass value="5.0"/>
-        <inertia ixx="0"  ixy="0"  ixz="0" iyy="0" iyz="0" izz="0" />
+        <mass value="4.8"/>
+        <inertia ixx="3.32e-2"  ixy="2.7e-6"  ixz="-3.3e-6" iyy="1.43e-2" iyz="2.3e-4" izz="2.54e-2" />
       </inertial>
       <visual>
@@ -163,7 +164,6 @@
     <link name="${prefix}link_4">
       <inertial>
-        <origin xyz="-0.00008 0.06528 0.06149" rpy="0 0 0"/>
-        <mass value="0.7"/>
-        <inertia ixx="0"  ixy="0"  ixz="0" iyy="0" iyz="0" izz="0" />
+        <mass value="0.9"/>
+        <inertia ixx="4.7e-2"  ixy="-1.1e-6"  ixz="-9.8e-6" iyy="4.15e-2" iyz="1.35e-2" izz="6.63e-3" />
       </inertial>
       <visual>
@@ -197,7 +197,6 @@
     <link name="${prefix}link_5">
       <inertial>
-        <origin xyz="-0.00026 0.01873 -0.03434" rpy="0 0 0"/>
-        <mass value="2"/>
-        <inertia ixx="0"  ixy="0"  ixz="0" iyy="0" iyz="0" izz="0" />
+        <mass value="2.6"/>
+        <inertia ixx="1.13e-2"  ixy="6.0e-5"  ixz="-2.7e-5" iyy="8.68e-3" iyz="7.9e-5" izz="5.10e-3" />
       </inertial>
       <visual>
@@ -249,4 +248,8 @@
     <!-- Flange -->
     <link name="${prefix}flange">
+      <inertial>
+        <mass value="0.1" />
+        <inertia ixx="0" ixy="0" ixz="0" iyy="0" iyz="0" izz="0" />
+      </inertial>
       <visual>
         <origin xyz="0 0 0" rpy="0 0 0" />
@@ -276,4 +279,52 @@
       <child link="${prefix}tool0" />
     </joint>
+    <!-- transmissions for gazebo -->
+    <transmission name="${prefix}joint_1_trans">
+      <type>transmission_interface/SimpleTransmission</type>
+      <joint name="${prefix}joint_1">
+        <hardwareInterface>hardware_interface/PositionJointInterface</hardwareInterface>
+      </joint>
+      <actuator name="${prefix}joint_1_motor"/>
+    </transmission>
+    <transmission name="${prefix}joint_2_trans">
+      <type>transmission_interface/SimpleTransmission</type>
+      <joint name="${prefix}joint_2">
+        <hardwareInterface>hardware_interface/PositionJointInterface</hardwareInterface>
+      </joint>
+      <actuator name="${prefix}joint_2_motor"/>
+    </transmission>
+    <transmission name="${prefix}joint_3_trans">
+      <type>transmission_interface/SimpleTransmission</type>
+      <joint name="${prefix}joint_3">
+        <hardwareInterface>hardware_interface/PositionJointInterface</hardwareInterface>
+      </joint>
+      <actuator name="${prefix}joint_3_motor"/>
+    </transmission>
+    <transmission name="${prefix}joint_4_trans">
+      <type>transmission_interface/SimpleTransmission</type>
+      <joint name="${prefix}joint_4">
+        <hardwareInterface>hardware_interface/PositionJointInterface</hardwareInterface>
+      </joint>
+      <actuator name="${prefix}joint_4_motor"/>
+    </transmission>
+    <transmission name="${prefix}joint_5_trans">
+      <type>transmission_interface/SimpleTransmission</type>
+      <joint name="${prefix}joint_5">
+        <hardwareInterface>hardware_interface/PositionJointInterface</hardwareInterface>
+      </joint>
+      <actuator name="${prefix}joint_5_motor"/>
+    </transmission>
+    <transmission name="${prefix}joint_6_trans">
+      <type>transmission_interface/SimpleTransmission</type>
+      <joint name="${prefix}joint_6">
+        <hardwareInterface>hardware_interface/PositionJointInterface</hardwareInterface>
+      </joint>
+      <actuator name="${prefix}joint_6_motor"/>
+    </transmission>
+    <gazebo>
+      <plugin name="gazebo_ros_control" filename="libgazebo_ros_control.so" >
+        <robotNamespace>prbt</robotNamespace>
+      </plugin>
+    </gazebo>
   </xacro:macro>
 </robot>

Commit message: Fix name joint name

File: prbt_support/urdf/prbt.xacro (robot description, xacro)
@@ -31,5 +31,5 @@
   <xacro:prbt prefix="$(arg robot_prefix)" />
   <link name="world"/>
-  <joint name="fixed" type="fixed">
+  <joint name="world-base_link-fixed" type="fixed">
     <parent link="world"/>
     <child link="$(arg robot_prefix)base_link"/>

Commit message: swapped child and parent in world-base link

File: prbt_support/urdf/prbt.xacro (robot description, xacro)
@@ -32,6 +32,7 @@
   <link name="world"/>
   <joint name="world-base_link-fixed" type="fixed">
-    <parent link="world"/>
-    <child link="$(arg robot_prefix)base_link"/>
+    <child link="world"/>
+    <parent link="$(arg robot_prefix)base_link"/>
+    <origin xyz="0.0 0.0 0.0" rpy="0.0 0.0 0.0" />
   </joint>
   <!-- TCP -->

Commit message: Revert "swapped child and parent in world-base link"
This reverts commit 0ff1dde1e61d7fac53480f49b5f39f67b6bf244f.

File: prbt_support/urdf/prbt.xacro (robot description, xacro)
@@ -32,7 +32,6 @@
   <link name="world"/>
   <joint name="world-base_link-fixed" type="fixed">
-    <child link="world"/>
-    <parent link="$(arg robot_prefix)base_link"/>
-    <origin xyz="0.0 0.0 0.0" rpy="0.0 0.0 0.0" />
+    <parent link="world"/>
+    <child link="$(arg robot_prefix)base_link"/>
   </joint>
   <!-- TCP -->

Commit message: gripper brackets configurable
* no longer require parent_left and parent_right arguments, but set
  default values from the gripper name
* add optional parameters to configure the size of the brackets

File: prbt_support/urdf/prbt.xacro (robot description, xacro)
@@ -49,8 +49,5 @@
     <!-- Add gripper brackets -->
     <xacro:include filename="$(find prbt_support)/urdf/simple_gripper_brackets.urdf.xacro" />
-    <xacro:simple_gripper_brackets
-        gripper_name="$(arg gripper_name)"
-        parent_left="$(arg gripper_name)_finger_left_link"
-        parent_right="$(arg gripper_name)_finger_right_link"/>
+    <xacro:simple_gripper_brackets gripper_name="$(arg gripper_name)" />
   </xacro:if>
 </robot>

File: prbt_support/urdf/simple_gripper_brackets.urdf.xacro (robot description, xacro)
@@ -13,5 +13,17 @@
 -->
 <robot xmlns:xacro="http://www.ros.org/wiki/xacro">
-  <xacro:macro name="simple_gripper_brackets" params="gripper_name parent_left parent_right">
+  <xacro:macro name="simple_gripper_brackets"
+               params="gripper_name
+                       parent_left:=^|''
+                       parent_right:=^|''
+                       size_x:=^|0.03
+                       size_y:=^|0.01
+                       size_z:=^|0.05">
+    <xacro:if value="${parent_left==''}">
+      <xacro:property name="parent_left" value="${gripper_name}_finger_left_link" />
+    </xacro:if>
+    <xacro:if value="${parent_right==''}">
+      <xacro:property name="parent_right" value="${gripper_name}_finger_right_link" />
+    </xacro:if>
     <!-- fixed joint attaching to left bracket mounting -->
     <joint name="${gripper_name}_link_left_bracket_fixed_joint" type="fixed">
@@ -27,7 +39,7 @@
         </inertial>
         <visual>
-          <origin xyz="0 0.005 0.02" rpy="0 0 0" />
+          <origin xyz="0 ${size_y/2} ${size_z/2-0.005}" rpy="0 0 0" />
           <geometry>
-            <box size="0.03 0.01 0.05"/>
+            <box size="${size_x} ${size_y} ${size_z}"/>
           </geometry>
           <material name="light_gray">
@@ -36,7 +48,7 @@
         </visual>
         <collision>
-          <origin xyz="0 0.005 0.02" rpy="0 0 0" />
+          <origin xyz="0 ${size_y/2} ${size_z/2-0.005}" rpy="0 0 0" />
           <geometry>
-            <box size="0.03 0.01 0.05"/>
+            <box size="${size_x} ${size_y} ${size_z}"/>
           </geometry>
         </collision>
@@ -55,7 +67,7 @@
         </inertial>
         <visual>
-          <origin xyz="0 -0.005 0.02" rpy="0 0 0" />
+          <origin xyz="0 -${size_y/2} ${size_z/2-0.005}" rpy="0 0 0" />
           <geometry>
-            <box size="0.03 0.01 0.05"/>
+            <box size="${size_x} ${size_y} ${size_z}"/>
           </geometry>
           <material name="dark_grey">
@@ -64,7 +76,7 @@
         </visual>
         <collision>
-          <origin xyz="0 -0.005 0.02" rpy="0 0 0" />
+          <origin xyz="0 -${size_y/2} ${size_z/2-0.005}" rpy="0 0 0" />
           <geometry>
-            <box size="0.03 0.01 0.05"/>
+            <box size="${size_x} ${size_y} ${size_z}"/>
           </geometry>
         </collision>

Commit message: allow gripper_name as outside property
instead of passing it explicitly

File: prbt_support/urdf/prbt.xacro (robot description, xacro)
@@ -45,9 +45,9 @@
   <xacro:if value="${gripper != ''}">
     <!-- name of the gripper -->
-    <xacro:arg name="gripper_name" default="$(arg robot_prefix)gripper"/>
+    <xacro:property name="gripper_name" value="$(arg robot_prefix)gripper"/>
     <xacro:include filename="$(find prbt_${gripper}_support)/urdf/${gripper}.urdf.xacro" />
     <!-- Add gripper brackets -->
     <xacro:include filename="$(find prbt_support)/urdf/simple_gripper_brackets.urdf.xacro" />
-    <xacro:simple_gripper_brackets gripper_name="$(arg gripper_name)" />
+    <xacro:simple_gripper_brackets />
   </xacro:if>
 </robot>

File: prbt_support/urdf/simple_gripper_brackets.urdf.xacro (robot description, xacro)
@@ -14,5 +14,5 @@
 <robot xmlns:xacro="http://www.ros.org/wiki/xacro">
   <xacro:macro name="simple_gripper_brackets"
-               params="gripper_name
+               params="gripper_name:=^
                        parent_left:=^|''
                        parent_right:=^|''

Commit message: preparing kinetic merge

File: prbt_support/urdf/prbt.xacro (robot description, xacro)
@@ -44,5 +44,10 @@
   <!-- If gripper given then... -->
   <xacro:if value="${gripper != ''}">
+    <!-- name of the gripper -->
+    <xacro:property name="gripper_name" value="$(arg robot_prefix)gripper"/>
     <xacro:include filename="$(find prbt_${gripper}_support)/urdf/${gripper}.urdf.xacro" />
+    <!-- Add gripper brackets -->
+    <xacro:include filename="$(find prbt_support)/urdf/simple_gripper_brackets.urdf.xacro" />
+    <xacro:simple_gripper_brackets />
   </xacro:if>
 </robot>

File: prbt_support/urdf/simple_gripper_brackets.urdf.xacro (robot description, xacro)
@@ -13,5 +13,17 @@
 -->
 <robot xmlns:xacro="http://www.ros.org/wiki/xacro">
-  <xacro:macro name="simple_gripper_brackets" params="gripper_name parent_left parent_right">
+  <xacro:macro name="simple_gripper_brackets"
+               params="gripper_name:=^
+                       parent_left:=^|''
+                       parent_right:=^|''
+                       size_x:=^|0.03
+                       size_y:=^|0.01
+                       size_z:=^|0.05">
+    <xacro:if value="${parent_left==''}">
+      <xacro:property name="parent_left" value="${gripper_name}_finger_left_link" />
+    </xacro:if>
+    <xacro:if value="${parent_right==''}">
+      <xacro:property name="parent_right" value="${gripper_name}_finger_right_link" />
+    </xacro:if>
     <!-- fixed joint attaching to left bracket mounting -->
     <joint name="${gripper_name}_link_left_bracket_fixed_joint" type="fixed">
@@ -27,7 +39,7 @@
         </inertial>
         <visual>
-          <origin xyz="0 0.005 0.02" rpy="0 0 0" />
+          <origin xyz="0 ${size_y/2} ${size_z/2-0.005}" rpy="0 0 0" />
           <geometry>
-            <box size="0.03 0.01 0.05"/>
+            <box size="${size_x} ${size_y} ${size_z}"/>
           </geometry>
           <material name="light_gray">
@@ -36,7 +48,7 @@
         </visual>
         <collision>
-          <origin xyz="0 0.005 0.02" rpy="0 0 0" />
+          <origin xyz="0 ${size_y/2} ${size_z/2-0.005}" rpy="0 0 0" />
           <geometry>
-            <box size="0.03 0.01 0.05"/>
+            <box size="${size_x} ${size_y} ${size_z}"/>
           </geometry>
         </collision>
@@ -55,7 +67,7 @@
         </inertial>
         <visual>
-          <origin xyz="0 -0.005 0.02" rpy="0 0 0" />
+          <origin xyz="0 -${size_y/2} ${size_z/2-0.005}" rpy="0 0 0" />
           <geometry>
-            <box size="0.03 0.01 0.05"/>
+            <box size="${size_x} ${size_y} ${size_z}"/>
           </geometry>
           <material name="dark_grey">
@@ -64,7 +76,7 @@
         </visual>
         <collision>
-          <origin xyz="0 -0.005 0.02" rpy="0 0 0" />
+          <origin xyz="0 -${size_y/2} ${size_z/2-0.005}" rpy="0 0 0" />
           <geometry>
-            <box size="0.03 0.01 0.05"/>
+            <box size="${size_x} ${size_y} ${size_z}"/>
           </geometry>
         </collision>
