Commit message: fake frames to observe

File: prbt_hardware_support/test/config/speed_observer_test.xacro (robot description, xacro)
@@ -12,17 +12,19 @@
 limitations under the License.
 -->
-<robot name="prbt" xmlns:xacro="http://www.ros.org/wiki/xacro">
+<robot name="testing" xmlns:xacro="http://www.ros.org/wiki/xacro">
   <!-- Definition of robot name -->
   <xacro:arg name="robot_prefix" default="testing_"/>
   <link name="world"/>
   <joint name="$(arg robot_prefix)world-a" type="fixed">
+  <origin xyz="0 0 1" rpy="1.57079632679 0 0" />
     <parent link="world"/>
     <child link="$(arg robot_prefix)a"/>
   </joint>
   <link name="$(arg robot_prefix)a" />
-  <joint name="$(arg robot_prefix)a-b" type="fixed">
-    <origin xyz="0 0 0" rpy="0 0 0" />
-    <parent link="$(arg robot_prefix)a"/>
-    <child link="$(arg robot_prefix)b"/>
+  <joint name="$(arg robot_prefix)a-b" type="continuous">
+    <origin xyz="1 0 0" rpy="1.57079632679 0 0" />
+    <parent link="$(arg robot_prefix)a" />
+    <child link="$(arg robot_prefix)b" />
+    <limit effort="999" velocity="99" />
   </joint>
   <link name="$(arg robot_prefix)b" />

Commit message: a working xacro model and spinner in test

File: prbt_hardware_support/test/config/speed_observer_test.xacro (robot description, xacro)
@@ -16,15 +16,15 @@
   <xacro:arg name="robot_prefix" default="testing_"/>
   <link name="world"/>
-  <joint name="$(arg robot_prefix)world-a" type="fixed">
-  <origin xyz="0 0 1" rpy="1.57079632679 0 0" />
+  <joint name="$(arg robot_prefix)world-a" type="continuous">
+  <origin xyz="0 0 1" rpy="0 1.57079632679 0" />
     <parent link="world"/>
     <child link="$(arg robot_prefix)a"/>
+    <limit effort="999" velocity="99" />
   </joint>
   <link name="$(arg robot_prefix)a" />
-  <joint name="$(arg robot_prefix)a-b" type="continuous">
-    <origin xyz="1 0 0" rpy="1.57079632679 0 0" />
+  <joint name="$(arg robot_prefix)a-b" type="fixed">
+    <origin xyz="0 1 0" rpy="0 0 0" />
     <parent link="$(arg robot_prefix)a" />
     <child link="$(arg robot_prefix)b" />
-    <limit effort="999" velocity="99" />
   </joint>
   <link name="$(arg robot_prefix)b" />

Commit message: Update prbt_hardware_support/test/config/speed_observer_test.xacro
Co-Authored-By: Alexander Gutenkunst <a.gutenkunst@pilz.de>

File: prbt_hardware_support/test/config/speed_observer_test.xacro (robot description, xacro)
@@ -17,5 +17,5 @@
   <link name="world"/>
   <joint name="$(arg robot_prefix)world-a" type="continuous">
-  <origin xyz="0 0 1" rpy="0 1.57079632679 0" />
+  <origin xyz="0 0 1" rpy="0 ${pi/2} 0" />
     <parent link="world"/>
     <child link="$(arg robot_prefix)a"/>
