Commit message: Refator robot_mock model

File: pilz_control/test/urdf/robot_mock.urdf (robot description, URDF)
Before this commit: robot robot_mock, 2 links, 1 joints
Links:
- removed link link1
- removed link link2
- added link arm_left_link; visual cylinder length=0.125 radius=0.02
- added link arm_right_link; visual cylinder length=0.25 radius=0.05
- added link base_link; visual box size=0.3 0.1 0.5
- added link hand_left_link; visual box size=0.03 0.03 0.125
- added link hand_right_link; visual box size=0.05 0.05 0.25
- added link shoulder_link
Joints:
- removed joint joint1
- added joint arm_left_to_hand_left: type fixed, parent arm_left_link, child hand_left_link, origin xyz=0 0 0.125
- added joint arm_right_to_hand_right: type fixed, parent arm_right_link, child hand_right_link, origin xyz=0 0 0.25
- added joint base_to_shoulder: type fixed, parent base_link, child shoulder_link, origin xyz=0 0 0.25
- added joint shoulder_to_left_arm: type continuous, parent shoulder_link, child arm_left_link, origin xyz=0 -0.125 0, axis 0 1 0
- added joint shoulder_to_right_arm: type continuous, parent shoulder_link, child arm_right_link, origin xyz=0 0.25 0, axis 0 1 0

Commit message: Add end effector group to robot mock

File: pilz_control/test/urdf/robot_mock.urdf (robot description, URDF)
Before this commit: robot robot_mock, 6 links, 5 joints
Links:
- added link finger_right_link; visual box size=0.05 0.05 0.05
Joints:
- added joint hand_right_to_finger_right: type fixed, parent hand_right_link, child finger_right_link, origin xyz=0 0 0.025

Commit message: Add Cartesian speed monitoring

File: pilz_control/test/urdf/robot_mock.urdf (robot description, URDF)
Before this commit: robot robot_mock, 2 links, 1 joints
Links:
- removed link link1
- removed link link2
- added link arm_left_link; visual cylinder length=0.125 radius=0.02
- added link arm_right_link; visual cylinder length=0.25 radius=0.05
- added link base_link; visual box size=0.3 0.1 0.5
- added link finger_right_link; visual box size=0.05 0.05 0.05
- added link hand_left_link; visual box size=0.03 0.03 0.125
- added link hand_right_link; visual box size=0.05 0.05 0.25
- added link shoulder_link
Joints:
- removed joint joint1
- added joint arm_left_to_hand_left: type fixed, parent arm_left_link, child hand_left_link, origin xyz=0 0 0.125
- added joint arm_right_to_hand_right: type fixed, parent arm_right_link, child hand_right_link, origin xyz=0 0 0.25
- added joint base_to_shoulder: type fixed, parent base_link, child shoulder_link, origin xyz=0 0 0.25
- added joint hand_right_to_finger_right: type fixed, parent hand_right_link, child finger_right_link, origin xyz=0 0 0.025
- added joint shoulder_to_left_arm: type continuous, parent shoulder_link, child arm_left_link, origin xyz=0 -0.125 0, axis 0 1 0
- added joint shoulder_to_right_arm: type continuous, parent shoulder_link, child arm_right_link, origin xyz=0 0.25 0, axis 0 1 0
